File: hardware/balance-bot/balance-bot.kicad_pcb (KiCad board)
At the start: 2 copper layers, 95 x 75 mm, 25 parts, among them J1 Conn_01x15_Socket, J11 Conn_01x05_Pin, J12 Conn_01x04_Pin, J13 Conn_01x04_Pin, J2 Conn_01x15_Socket, J3 Conn_01x08_Socket, J4 Conn_01x04_Socket, J5 Conn_01x04_Socket, J6 Conn_01x03_Pin, J7 Conn_01x04_Socket, J8 Conn_01x02_Pin, J9 Conn_01x06_Pin, Q1 IRF4905, SW1 SW_SPDT

Commit message: PCB v1.0 Created 3d models and gerber files. Moved balancing step into its own module and set up pins for the encoders
Other:
- board text added: "IN+"
- board text added: "IN-"
Changed lines of the file:
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@@
 		(tenting front back)
 		(pcbplotparams
-			(layerselection 0x00000000_00000000_55555555_5755f5ff)
+			(layerselection 0x00000000_00000000_55555555_575555ff)
 			(plot_on_all_layers_selection 0x00000000_00000000_00000000_00000000)
 			(disableapertmacros no)
-			(usegerberextensions no)
+			(usegerberextensions yes)
 			(usegerberattributes yes)
 			(usegerberadvancedattributes yes)
@@
 			(sketchdnponfab yes)
 			(crossoutdnponfab yes)
-			(subtractmaskfromsilk no)
+			(subtractmaskfromsilk yes)
 			(outputformat 1)
 			(mirror no)
-			(drillshape 1)
+			(drillshape 0)
 			(scaleselection 1)
-			(outputdirectory "")
+			(outputdirectory "gerbers/")
 		)
 	)
@@
 		(layer "F.SilkS")
 		(effects
+			(font
+				(size 1 1)
+				(thickness 0.1)
+			)
+			(justify left bottom)
+		)
+	)
+	(gr_text "IN-"
+		(at 40.5 76 0)
+		(layer "F.SilkS")
+		(effects
+			(font
+				(size 1 1)
+				(thickness 0.1)
+			)
+			(justify left bottom)
+		)
+	)
+	(gr_text "IN+"
+		(at 58 76 0)
+		(layer "F.SilkS")
+		(effects
